Commit message: Выполнена лабораторная работа 3

File: src/myrobot/myrobot_description/urdf/myrobot.xacro (robot description, xacro)
@@ -5,5 +5,5 @@
   <xacro:property name="base_size_y" value="0.3"/>
   <xacro:property name="base_size_z" value="0.1"/>
-  <xacro:property name="base_mass" value="5"/>
+  <xacro:property name="base_mass" value="0.1"/>
   <xacro:property name="wheel_radius" value="0.05"/>
   <xacro:property name="wheel_width" value="0.025"/>
@@ -19,5 +19,5 @@
   <xacro:property name="base_y" value="0.0"/>
   <xacro:property name="base_z" value="${wheel_radius}"/>
-  <xacro:property name="wheel_base_x" value="${-wheel_radius}"/>
+  <xacro:property name="wheel_base_x" value="0.0"/>
   <xacro:property name="wheel_base_y" value="${base_size_y / 2 + wheel_width / 2}"/>
   <xacro:property name="wheel_base_z" value="0.0"/>
@@ -58,4 +58,7 @@
       <origin xyz="${roller_base_x} ${roller_base_y} ${roller_base_z}"/>
     </xacro:roller>
+    <xacro:roller name="back" parent="base_link" radius="${roller_radius}" mass="${roller_mass}">
+      <origin xyz="${-roller_base_x} ${roller_base_y} ${roller_base_z}"/>
+    </xacro:roller>
     <!-- ============ Enter sensors code here =============== -->
     <!-- ============ LIDAR =============== -->

File: src/myrobot/myrobot_simulator/urdf/macro.gazebo.xacro (robot description, xacro)
@@ -2,14 +2,18 @@
 <robot xmlns:xacro="http://www.ros.org/wiki/xacro">
   <gazebo reference="left_wheel">
-    <mu1>4</mu1>
-    <mu2>4</mu2>
+    <mu1>5</mu1>
+    <mu2>5</mu2>
   </gazebo>
   <gazebo reference="right_wheel">
-    <mu1>4</mu1>
-    <mu2>4</mu2>
+    <mu1>5</mu1>
+    <mu2>5</mu2>
   </gazebo>
   <gazebo reference="front_roller">
-    <mu1>0</mu1>
-    <mu2>0</mu2>
+    <mu1>0.1</mu1>
+    <mu2>0.1</mu2>
+  </gazebo>
+  <gazebo reference="back_roller">
+    <mu1>0.1</mu1>
+    <mu2>0.1</mu2>
   </gazebo>
   <gazebo reference="base_link">
